File: basic_mxm_nvme/basic_mxm_nvme.kicad_pcb (KiCad board)
At the start: 2 copper layers, 82 x 61.8 mm, 6 parts, among them CN1 AS0B826-S78B-7H, J1 Bus_M.2_Socket_M, J2 Bus_M.2_Socket_M, J3 Bus_M.2_Socket_M

Commit message: Added clock buffer to schematic
and put the footprints in the pcb file
Parts:
- added C1: 100nF, Capacitor_SMD:C_0603_1608Metric, F.Cu at (27.1, 107.0)
- added C2: 100nF, Capacitor_SMD:C_0603_1608Metric, F.Cu at (27.1, 109.5)
- added C3: 100nF, Capacitor_SMD:C_0603_1608Metric, F.Cu at (27.1, 112.0)
- added C4: 100nF, Capacitor_SMD:C_0603_1608Metric, F.Cu at (27.1, 114.5)
- added C5: 100nF, Capacitor_SMD:C_0603_1608Metric, F.Cu at (27.1, 117.1)
- added C6: 100nF, Capacitor_SMD:C_0603_1608Metric, F.Cu at (27.1, 119.6)
- added C7: 100nF, Capacitor_SMD:C_0603_1608Metric, F.Cu at (27.1, 122.1)
- added C8: 100nF, Capacitor_SMD:C_0603_1608Metric, F.Cu at (31.2, 107.0)
- added C9: 100nF, Capacitor_SMD:C_0603_1608Metric, F.Cu at (31.2, 109.5)
- added H3: MountingHole_Pad, TestPoint:TestPoint_THTPad_D3.0mm_Drill1.5mm, F.Cu at (39.7, 123.2)
- added J4: qwiic, Connector_JST:JST_SH_SM04B-SRSS-TB_1x04-1MP_P1.00mm_Horizontal, F.Cu at (41.6, 109.6)
- added R1: 10kΩ, Resistor_SMD:R_0603_1608Metric, F.Cu at (31.2, 112.0)
- added R2: 10kΩ, Resistor_SMD:R_0603_1608Metric, F.Cu at (31.2, 114.5)
- added R3: 10kΩ, Resistor_SMD:R_0603_1608Metric, F.Cu at (31.2, 117.1)
- added R4: 10kΩ, Resistor_SMD:R_0603_1608Metric, F.Cu at (31.2, 119.6)
- added R5: 10kΩ, Resistor_SMD:R_0603_1608Metric, F.Cu at (31.2, 122.1)
- added R6: 10kΩ, Resistor_SMD:R_0603_1608Metric, F.Cu at (35.2, 107.0)
- added R7: 10kΩ, Resistor_SMD:R_0603_1608Metric, F.Cu at (35.2, 109.5)
- added R8: 10kΩ, Resistor_SMD:R_0603_1608Metric, F.Cu at (35.2, 112.0)
- added R9: 10kΩ, Resistor_SMD:R_0603_1608Metric, F.Cu at (35.2, 114.5)
- added U1: clockbuffer_9ZXL0651AKLF, A-my-stuff:clockbuffer_9ZXL0651AKLF, F.Cu at (40.8, 117.0)
Connections:
- CN1 pad 153: unconnected-(CN1-PEX_REFCLK#-Pad153) -> Host_REFCLK-
- CN1 pad 154: unconnected-(CN1-PEX_CLK_REQ#-Pad154) -> GND
- CN1 pad 155: unconnected-(CN1-PEX_REFCLK-Pad155) -> Host_REFCLK+
- CN1 pad 156: unconnected-(CN1-PEX_RST#-Pad156) -> PERST#
- CN1 pad 4: unconnected-(CN1-WAKE#-Pad4) -> PEWAKE#
- J1 pad 50: unconnected-(J1-~{PERST}-Pad50) -> PERST#
- J1 pad 52: unconnected-(J1-~{CLKREQ}-Pad52) -> Slot1_CLKREQ#
- J1 pad 53: unconnected-(J1-REFCLKn-Pad53) -> Slot1_REFCLK-
- J1 pad 54: unconnected-(J1-~{PEWAKE}-Pad54) -> PEWAKE#
- J1 pad 55: unconnected-(J1-REFCLKp-Pad55) -> Slot1_REFCLK+
- J2 pad 50: unconnected-(J2-~{PERST}-Pad50) -> PERST#
- J2 pad 52: unconnected-(J2-~{CLKREQ}-Pad52) -> Slot2_CLKREQ#
- J2 pad 53: unconnected-(J2-REFCLKn-Pad53) -> Slot2_REFCLK-
- J2 pad 54: unconnected-(J2-~{PEWAKE}-Pad54) -> PEWAKE#
- J2 pad 55: unconnected-(J2-REFCLKp-Pad55) -> Slot2_REFCLK+
- J3 pad 50: unconnected-(J3-~{PERST}-Pad50) -> PERST#
- J3 pad 52: unconnected-(J3-~{CLKREQ}-Pad52) -> Slot3_CLKREQ#
- J3 pad 53: unconnected-(J3-REFCLKn-Pad53) -> Slot3_REFCLK-
- J3 pad 54: unconnected-(J3-~{PEWAKE}-Pad54) -> PEWAKE#
- J3 pad 55: unconnected-(J3-REFCLKp-Pad55) -> Slot3_REFCLK+
Routing:
- added copper zone on B.Cu, net PERST#
- added copper zone on F.Cu, net PERST#
- removed copper zone on B.Cu, net GND
- removed copper zone on F.Cu, net GND
