File: basic_mxm_nvme/basic_mxm_nvme.kicad_sch (KiCad schematic)
At the start: 6 parts, among them CN1 AS0B826-S78B-7H, J1 Bus_M.2_Socket_M, J2 Bus_M.2_Socket_M, J3 Bus_M.2_Socket_M

Commit message: Added clock buffer to schematic
and put the footprints in the pcb file
Parts:
- added C1, C2, C3, C4, C5, C6, C7, C8, C9: 100nF, Capacitor_SMD:C_0603_1608Metric, symbol Device:C_Small
- added H3: MountingHole_Pad, TestPoint:TestPoint_THTPad_D3.0mm_Drill1.5mm, symbol Mechanical:MountingHole_Pad
- added J4: qwiic, Connector_JST:JST_SH_SM04B-SRSS-TB_1x04-1MP_P1.00mm_Horizontal, symbol Connector_Generic_MountingPin:Conn_01x04_MountingPin
- added R1, R2, R3, R4, R5, R6, R7, R8, R9: 10kΩ, Resistor_SMD:R_0603_1608Metric, symbol Device:R_Small
- added U1: clockbuffer_9ZXL0651AKLF, A-my-stuff:clockbuffer_9ZXL0651AKLF, symbol A-my-stuff:clockbuffer_9ZXL0651AKLF
Connections:
- net GND: now also CN1.154 (PEX_CLK_REQ#), C1.2, C2.2, C3.2, C4.2, C5.2, C6.2, C7.2, C8.2, C9.2, H3.1, J4.1 (Pin_1), J4.MP (MountPin), R5.2, U1.4 (GND_1), U1.41 (GND_2)
- net Host_REFCLK-: now reaches CN1.153 (PEX_REFCLK#)
- net Host_REFCLK-: now also U1.7 (DIF_IN#)
- net Host_REFCLK+: now reaches CN1.155 (PEX_REFCLK)
- net Host_REFCLK+: now also U1.6 (DIF_IN)
- net PERST#: now reaches CN1.156 (PEX_RST#)
- net PERST#: now also J1.50 (~{PERST}), J2.50 (~{PERST}), J3.50 (~{PERST})
- net PEWAKE#: now reaches CN1.4 (WAKE#)
- net PEWAKE#: now also J1.54 (~{PEWAKE}), J2.54 (~{PEWAKE}), J3.54 (~{PEWAKE})
- net Slot3_CLKREQ#: now reaches J3.52 (~{CLKREQ})
- net Slot3_CLKREQ#: now also R9.2, U1.22 (vOE2#)
- net Slot3_REFCLK-: now reaches J3.53 (REFCLKn)
- net Slot3_REFCLK-: now also U1.24 (DIF_2#)
- net Slot3_REFCLK+: now reaches J3.55 (REFCLKp)
- net Slot3_REFCLK+: now also U1.23 (DIF_2)
- net Slot1_CLKREQ#: now reaches J1.52 (~{CLKREQ})
- net Slot1_CLKREQ#: now also R6.2, U1.13 (vOE0#)
- net Slot1_REFCLK-: now reaches J1.53 (REFCLKn)
- net Slot1_REFCLK-: now also U1.15 (DIF_0#)
- net Slot1_REFCLK+: now reaches J1.55 (REFCLKp)
- net Slot1_REFCLK+: now also U1.14 (DIF_0)
- net Slot2_CLKREQ#: now reaches J2.52 (~{CLKREQ})
- net Slot2_CLKREQ#: now also R7.2, U1.19 (vOE1#)
- net Slot2_REFCLK-: now reaches J2.53 (REFCLKn)
- net Slot2_REFCLK-: now also U1.18 (DIF_1#)
- net Slot2_REFCLK+: now reaches J2.55 (REFCLKp)
- net Slot2_REFCLK+: now also U1.17 (DIF_1)
- new net: R4.2, R5.1, U1.2 (^vHIBW_BYPM_LOBW#)
- new net: R8.2, U1.28 (vOE3#), U1.32 (vOE4#), U1.38 (vOE5#)
- new net: R2.2, U1.3 (CKPWRGD_PD#)
- new net +3.3V: C1.1, C2.1, C3.1, C4.1, C5.1, C6.1, C7.1, C8.1, C9.1, J4.2 (Pin_2), R1.1, R2.1, R3.1, R4.1, R6.1, R7.1, R8.1, R9.1, U1.1 (VDDA), U1.12 (VDD_1), U1.16 (VDD_2), U1.20 (VDD_3), U1.21 (VDD_4), U1.25 (VDD_5), U1.29 (VDD_6), U1.31 (VDD_7), U1.35 (VDD_8), U1.39 (VDD_9), U1.5 (VDDR)
- new net Buffer_SMBus_CLK: J4.4 (Pin_4), R3.2, U1.9 (SMBCLK)
- new net Buffer_SMBus_DAT: J4.3 (Pin_3), R1.2, U1.8 (SMBDAT)
- no-connect marks 0 -> 4
